Commit message: add visualization and plot function in papers

File: datasets/assets/UR5+gripper/ur5_gripper.urdf (robot description, URDF)
Before this commit: robot ur5, 52 links, 51 joints
Links:
- added link task_tcp
- added link task_tool_link, mass 0.008; collision cylinder length=0.032 radius=0.0045; collision cylinder length=0.087 radius=0.0036
- link box_link: geometry visual box size=.42 .28 0.87
Joints:
- added joint gripperpalm-task_tool_fixed_joint: type fixed, parent gripperpalm, child task_tool_link, origin xyz=0 0.055 0 rpy=0 0 1.570796325
- added joint task_tool-task_tcp_fixed_joint: type fixed, parent task_tool_link, child task_tcp, origin xyz=0.035 0 0 rpy=0 0 0
- joint shoulder_lift_joint: limit lower=-3.14159265 upper=-0.9 effort=150.0 velocity=3.15 -> lower=-3.14159265 upper=3.14159265 effort=150.0 velocity=3.15
